File: erie_rov_connector_board/erie_rov_connector_board.kicad_pcb (KiCad board)
At the start: 2 copper layers, 114.3 x 127 mm, 27 parts, among them J1 1761426-1, J10 CAM, J11 OSD, J12 VTX, J13 STRB, J14 Expansion, J2 PANEL, J3 BATT, J4 LOAD, J5 Thruster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

Commit message: Final changes before ordering v1.0
Other:
- board text added: "Connector Board The Erie ROV Project v0.1 2025-15-03"
- board text added: "Noah Mollerstuen Amitan Bar-Evan Mikael Steinman Gary Bailey"
