File: erie_rov_mainboard/erie_rov_mainboard.kicad_pcb (KiCad board)
At the start: 2 copper layers, 88.5 x 94 mm, 32 parts, among them J1 1761426-1, J10 Telem2-Teensy, J11 I2C, J12 GPS, J13 SERIAL4/5-OSD, J14 Rudder, J15 Expansion, J2 BATT, J3 CC PANEL, J4 CC BATT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

Commit message: Final changes before ordering v1.0
Parts:
- added C6: 10n, Capacitor_SMD:C_0805_2012Metric_Pad1.18x1.45mm_HandSolder, F.Cu at (84.5, 192.2)
- added R6: 1k, Resistor_SMD:R_0805_2012Metric_Pad1.20x1.40mm_HandSolder, F.Cu at (86.1, 189.2)
- C1, C2, C3, C4, C5: footprint CC0805KRX7R9BB104:CC0805N_YAG -> Capacitor_SMD:C_0805_2012Metric_Pad1.18x1.45mm_HandSolder
- J9: value TELEM1-Radio -> Telem1-Radio
- Q1, Q2, Q3: footprint digikey-footprints:SOT-23-3 -> Package_TO_SOT_SMD:SOT-23_Handsoldering
- R1, R3: footprint CRG0805F100R:RES0805_CRG_TYCO_TYC -> Resistor_SMD:R_0805_2012Metric_Pad1.20x1.40mm_HandSolder
- R2, R4, R5: footprint CRGCQ0805F10K:RESC2012X65N -> Resistor_SMD:R_0805_2012Metric_Pad1.20x1.40mm_HandSolder
- U2: footprint MAX3232CUE_T:21-0066-J_16L_MXM -> Package_SO:TSSOP-16_4.4x5mm_P0.65mm
- moved Q2 3.69 mm to (86.4, 185.4)
- moved R3 3.33 mm to (89.9, 183.4)
- moved R4 3.31 mm to (91.9, 183.4)
- moved C3 1.27 mm to (64.8, 150.5)
- moved C1 1.02 mm to (64.8, 152.7)
- moved C2 0.76 mm to (64.8, 154.8)
- moved C4 0.51 mm to (64.8, 157.0)
- moved R1 0.37 mm to (135.9, 188.5)
- moved R2 0.34 mm to (138.4, 188.5)
- moved R5 0.25 mm to (92.1, 193.4)
- moved Q1 0.16 mm to (136.9, 193.2)
Connections:
- Q3 pad 1: Net-(Q2-D) -> Net-(Q3-G)
- R5 pad 2: Net-(Q2-D) -> Net-(Q3-G)
Routing:
- net Net-(Q3-G): track 0.00 -> 11.1 mm
- net Net-(Q2-D): track 8.31 -> 2.62 mm
- net VTX_SW: track 6.91 -> 3.31 mm
- net GND: track 198.5 -> 201.6 mm, vias 78 -> 74
- net VID_PWR: track 5.61 -> 8.16 mm
- net RDR_PWM: track 68.5 -> 70.6 mm
- net LOAD_CC: track 110.9 -> 110.0 mm
- net TELEM_GND: track 8.81 -> 8.20 mm
- net Net-(U2-C2+): track 4.72 -> 5.24 mm
Other:
- board text added: "Main Board The Erie ROV Project v0.1 2025-15-03"
- board text added: "Noah Mollerstuen Amitan Bar-Evan Mikael Steinman Gary Bailey"
